Commit message: Deleted roblochon_gazebo. Replache roBLOchon by roBOchon.

File: robochon_description/urdf/robochon.urdf.xacro (robot description, xacro)
@@ -1,22 +1,34 @@
 <?xml version="1.0"?>
-<robot name="mimi" xmlns:xacro="http://ros.org/wiki/xacro">
+<robot name="robochon" xmlns:xacro="http://ros.org/wiki/xacro">
   <!-- Define robot constants -->
-  <xacro:property name="base_width" value="0.31"/>
-  <xacro:property name="base_length" value="0.42"/>
-  <xacro:property name="base_height" value="0.18"/>
-  <xacro:property name="wheel_radius" value="0.10"/>
-  <xacro:property name="wheel_width" value="0.04"/>
-  <xacro:property name="wheel_ygap" value="0.025"/>
-  <xacro:property name="wheel_zoff" value="0.05"/>
-  <xacro:property name="wheel_xoff" value="0.12"/>
-  <xacro:property name="caster_xoff" value="0.14"/>
+  <xacro:property name="base_width" value="${3*0.31}" />
+  <xacro:property name="base_length" value="${3*0.42}" />
+  <xacro:property name="base_height" value="0.18" />
+  <xacro:property name="wheel_radius" value="0.20" />
+  <xacro:property name="wheel_width" value="0.04" />
+  <xacro:property name="wheel_ygap" value="0.025" />
+  <xacro:property name="wheel_zoff" value="0.1" />
+  <xacro:property name="wheel_xoff" value="0.36" />
+  <xacro:property name="caster_radius" value="${(wheel_radius+wheel_zoff-(base_height/2))}" />
+  <xacro:property name="caster_xoff" value="${base_length/3}" />
+  <!-- <xacro:property name="caster_xoff" value="${0.9*base_length/2}" /> -->
   <xacro:property name="camera" value="0.05" /> <!-- Size of square 'camera' box -->
   <xacro:property name="axel_offset" value="0.1" />
+  <xacro:property name="gripper_width" value="0.04" />
+  <xacro:property name="gripper_length" value="2." />
+  <xacro:property name="gripper_height" value="${(wheel_radius+wheel_zoff)/2}" />
   <!-- Define intertial property macros  -->
   <xacro:macro name="box_inertia" params="m w h d">
     <inertial>
-      <origin xyz="0 0 0" rpy="${pi/2} 0 ${pi/2}"/>
-      <mass value="${m}"/>
-      <inertia ixx="${(m/12) * (h*h + d*d)}" ixy="0.0" ixz="0.0" iyy="${(m/12) * (w*w + d*d)}" iyz="0.0" izz="${(m/12) * (w*w + h*h)}"/>
+      <origin xyz="0 0 0" rpy="${pi/2} 0 ${pi/2}" />
+      <mass value="${m}" />
+      <inertia ixx="${(m/12) * (h*h + d*d)}" ixy="0.0" ixz="0.0" iyy="${(m/12) * (w*w + d*d)}" iyz="0.0" izz="${(m/12) * (w*w + h*h)}" />
+    </inertial>
+  </xacro:macro>
+  <xacro:macro name="gripper_inertia" params="m w h d">
+    <inertial>
+      <origin xyz="0 0 0" rpy="${pi/2} 0 ${pi/2}" />
+      <mass value="${m}" />
+      <inertia ixx="${(m/12) * (h*h + d*d)}" ixy="0.0" ixz="0.0" iyy="${(m/12) * (w*w + d*d)}" iyz="0.0" izz="${(m/12) * (w*w + h*h)}" />
     </inertial>
   </xacro:macro>
@@ -24,38 +36,38 @@
     <inertial>
       <origin xyz="0 0 0" rpy="${pi/2} 0 0" />
-      <mass value="${m}"/>
-      <inertia ixx="${(m/12) * (3*r*r + h*h)}" ixy = "0" ixz = "0" iyy="${(m/12) * (3*r*r + h*h)}" iyz = "0" izz="${(m/2) * (r*r)}"/>
+      <mass value="${m}" />
+      <inertia ixx="${(m/12) * (3*r*r + h*h)}" ixy="0" ixz="0" iyy="${(m/12) * (3*r*r + h*h)}" iyz="0" izz="${(m/2) * (r*r)}" />
     </inertial>
   </xacro:macro>
   <xacro:macro name="sphere_inertia" params="m r">
     <inertial>
-      <mass value="${m}"/>
-      <inertia ixx="${(2/5) * m * (r*r)}" ixy="0.0" ixz="0.0" iyy="${(2/5) * m * (r*r)}" iyz="0.0" izz="${(2/5) * m * (r*r)}"/>
+      <mass value="${m}" />
+      <inertia ixx="${(2/5) * m * (r*r)}" ixy="0.0" ixz="0.0" iyy="${(2/5) * m * (r*r)}" iyz="0.0" izz="${(2/5) * m * (r*r)}" />
     </inertial>
   </xacro:macro>
   <!-- Robot Base -->
-  <link name="map">
+  <link name="base_link">
     <visual>
-      <origin xyz="0 0 0" rpy="0 0 0"/>
-      <geometry>
-        <box size="${base_length} ${base_width} ${base_height}"/>
+      <origin xyz="0 0 0" rpy="0 0 0" />
+      <geometry>
+        <box size="${base_length} ${base_width} ${base_height}" />
       </geometry>
       <material name="Cyan">
-        <color rgba="0 1.0 1.0 1.0"/>
+        <color rgba="0 1.0 1.0 1.0" />
       </material>
     </visual>
     <collision>
       <geometry>
-        <box size="${base_length} ${base_width} ${base_height}"/>
+        <box size="${base_length} ${base_width} ${base_height}" />
       </geometry>
     </collision>
-    <xacro:box_inertia m="15" w="${base_width}" d="${base_length}" h="${base_height}"/>
+    <xacro:box_inertia m="15" w="${base_width}" d="${base_length}" h="${base_height}" />
   </link>
   <!-- Robot Footprint -->
-  <link name="base_footprint"/>
+  <link name="base_footprint" />
   <joint name="base_joint" type="fixed">
-    <parent link="map"/>
-    <child link="base_footprint"/>
-    <origin xyz="0.0 0.0 ${-(wheel_radius+wheel_zoff)}" rpy="0 0 0"/>
+    <parent link="base_link" />
+    <child link="base_footprint" />
+    <origin xyz="0.0 0.0 ${-(wheel_radius+wheel_zoff)}" rpy="0 0 0" />
   </joint>
   <!-- Wheels -->
@@ -63,101 +75,140 @@
     <link name="${prefix}_link">
       <visual>
-        <origin xyz="0 0 0" rpy="${pi/2} 0 0"/>
-        <geometry>
-            <cylinder radius="${wheel_radius}" length="${wheel_width}"/>
+        <origin xyz="0 0 0" rpy="${pi/2} 0 0" />
+        <geometry>
+          <cylinder radius="${wheel_radius}" length="${wheel_width}" />
         </geometry>
         <material name="Gray">
-          <color rgba="0.5 0.5 0.5 1.0"/>
+          <color rgba="0.5 0.5 0.5 1.0" />
         </material>
       </visual>
       <collision>
-        <origin xyz="0 0 0" rpy="${pi/2} 0 0"/>
-        <geometry>
-          <cylinder radius="${wheel_radius}" length="${wheel_width}"/>
+        <origin xyz="0 0 0" rpy="${pi/2} 0 0" />
+        <geometry>
+          <cylinder radius="${wheel_radius}" length="${wheel_width}" />
         </geometry>
         <surface>
-            <friction>
-              <ode>
-                <mu1>1.2</mu1>
-                <mu2>1.2</mu2>
-              </ode>
-            </friction>
-            <contact>
-              <ode>
-                <kp>500000.0</kp>
-                <kd>10.0</kd>
-                <max_vel>0.1</max_vel>
-                <min_depth>0.001</min_depth>
-              </ode>
-            </contact>
-          </surface>
+          <friction>
+            <ode>
+              <mu1>1.2</mu1>
+              <mu2>1.2</mu2>
+            </ode>
+          </friction>
+          <contact>
+            <ode>
+              <kp>500000.0</kp>
+              <kd>10.0</kd>
+              <max_vel>0.1</max_vel>
+              <min_depth>0.001</min_depth>
+            </ode>
+          </contact>
+        </surface>
       </collision>
-      <xacro:cylinder_inertia m="0.5" r="${wheel_radius}" h="${wheel_width}"/>
+      <xacro:cylinder_inertia m="0.5" r="${wheel_radius}" h="${wheel_width}" />
     </link>
     <joint name="${prefix}_joint" type="continuous">
-      <parent link="map"/>
-      <child link="${prefix}_link"/>
-      <origin xyz="${x_reflect*wheel_xoff} ${y_reflect*(base_width/2+wheel_ygap)} ${-wheel_zoff}" rpy="0 0 0"/>
-      <axis xyz="0 1 0"/>
+      <parent link="base_link" />
+      <child link="${prefix}_link" />
+      <origin xyz="${x_reflect*wheel_xoff} ${y_reflect*(base_width/2+wheel_ygap)} ${-wheel_zoff}" rpy="0 0 0" />
+      <axis xyz="0 1 0" />
     </joint>
   </xacro:macro>
   <xacro:wheel prefix="drivewhl_l" x_reflect="-1" y_reflect="1" />
   <xacro:wheel prefix="drivewhl_r" x_reflect="-1" y_reflect="-1" />
-  <!-- Caster Wheel -->
-  <link name="front_caster">
+  <xacro:macro name="front_caster" params="prefix y_reflect link_daddy">
+    <link name="front_caster_${prefix}">
+      <visual>
+        <geometry>
+          <sphere radius="${caster_radius}" />
+        </geometry>
+        <material name="Cyan">
+          <color rgba="0 1.0 1.0 1.0" />
+        </material>
+      </visual>
+      <collision>
+        <origin xyz="0 0 0" rpy="0 0 0" />
+        <geometry>
+          <sphere radius="${caster_radius}" />
+        </geometry>
+      </collision>
+      <xacro:sphere_inertia m="0.5" r="${caster_radius}" />
+    </link>
+    <gazebo reference="front_caster_${prefix}">
+      <mu1>0.01</mu1>
+      <mu2>0.01</mu2>
+      <visual>
+        <material>Gazebo/White</material>
+      </visual>
+    </gazebo>
+    <joint name="caster_joint_${prefix}" type="fixed">
+      <parent link="${link_daddy}" />
+      <child link="front_caster_${prefix}" />
+      <origin xyz="${caster_xoff} ${y_reflect*0.7*base_width/2} ${-(base_height/2)}" rpy="0 0 0" />
+    </joint>
+  </xacro:macro>
+  <xacro:front_caster prefix="front_left" link_daddy="base_link" y_reflect="1" />
+  <xacro:front_caster prefix="front_right" link_daddy="base_link" y_reflect="-1" />
+  <!-- Gripper -->
+  <xacro:macro name="gripper" params="prefix x_reflect y_reflect z_reflect z_rotation lenght_x link_daddy">
+    <link name="${prefix}_link">
+      <visual>
+        <origin xyz="0 0 0" rpy="0 0 0" />
+        <geometry>
+          <box size="${gripper_length*lenght_x} ${gripper_width} ${gripper_height}" />
+        </geometry>
+        <material name="Cyan">
+          <color rgba="0 1.0 1.0 1.0" />
+        </material>
+      </visual>
+      <collision>
+        <geometry>
+          <box size="${gripper_length*lenght_x} ${gripper_width} ${gripper_height}" />
+        </geometry>
+      </collision>
+      <xacro:gripper_inertia m="2" w="${gripper_width*lenght_x}" d="${gripper_length}" h="${gripper_height}" />
+    </link>
+    <gazebo reference="${prefix}_link">
+      <mu1>1.4</mu1>
+      <mu2>1.4</mu2>
+      <visual>
+        <material>Gazebo/White</material>
+      </visual>
+    </gazebo>
+    <joint name="${prefix}_joint" type="fixed">
+      <parent link="${link_daddy}" />
+      <child link="${prefix}_link" />
+      <origin xyz="${x_reflect*base_length/4} ${y_reflect*(base_width*0.6)} ${(-base_height/2 -wheel_zoff)*z_reflect}" rpy="0 0 ${z_rotation}" />
+    </joint>
+  </xacro:macro>
+  <xacro:gripper prefix="gripper_l" x_reflect="1" y_reflect="1" z_reflect="1" z_rotation="0.3" lenght_x="1" link_daddy="base_link" />
+  <xacro:gripper prefix="gripper_r" x_reflect="1" y_reflect="-1" z_reflect="1" z_rotation="-0.3" lenght_x="1" link_daddy="base_link" />
+  <xacro:gripper prefix="gripper_hor" x_reflect="-2" y_reflect="0" z_reflect="1" z_rotation="1.57" lenght_x="0.5" link_daddy="base_link" />
+  <xacro:gripper prefix="gripper_l_front" x_reflect="1.7" y_reflect="-0.45" z_reflect="0" z_rotation="0.5" lenght_x="0.5" link_daddy="gripper_l_link" />
+  <xacro:gripper prefix="gripper_r_front" x_reflect="1.7" y_reflect="0.45" z_reflect="0" z_rotation="-0.5" lenght_x="0.5" link_daddy="gripper_r_link" />
+  <!-- LIDAR -->
+  <joint name="lidar_joint" type="fixed">
+    <parent link="base_link" />
+    <child link="lidar_link" />
+    <origin xyz="${base_length/2} 0 0.115" rpy="0 0 0" />
+  </joint>
+  <link name="lidar_link">
     <visual>
-      <geometry>
-        <sphere radius="${(wheel_radius+wheel_zoff-(base_height/2))}"/>
-      </geometry>
-      <material name="Cyan">
-        <color rgba="0 1.0 1.0 1.0"/>
+      <origin xyz="0 0 0" rpy="0 0 0" />
+      <geometry>
+        <cylinder radius="0.0508" length="0.05" />
+      </geometry>
+      <material name="Black">
+        <color rgba="${0/255} ${0/255} ${0/255} 1.0" />
       </material>
     </visual>
     <collision>
-      <origin xyz="0 0 0" rpy="0 0 0"/>
-      <geometry>
-        <sphere radius="${(wheel_radius+wheel_zoff-(base_height/2))}"/>
+      <origin xyz="0 0 0" rpy="0 0 0" />
+      <geometry>
+        <cylinder radius="0.0508" length="0.05" />
       </geometry>
     </collision>
-    <xacro:sphere_inertia m="0.5" r="${(wheel_radius+wheel_zoff-(base_height/2))}"/>
-  </link>
-  <!-- Adding slippery mate5rial -->
-  <gazebo reference="front_caster">
-    <mu1>0.01</mu1>
-    <mu2>0.01</mu2>
-    <visual>
-      <material>Gazebo/White</material>
-    </visual>
-  </gazebo>
-  <joint name="caster_joint" type="fixed">
-    <parent link="map"/>
-    <child link="front_caster"/>
-    <origin xyz="${caster_xoff} 0.0 ${-(base_height/2)}" rpy="0 0 0"/>
-  </joint>
-  <!-- LIDAR -->
-  <joint name="lidar_joint" type="fixed">
-    <parent link="map"/>
-    <child link="lidar_link"/>
-    <origin xyz="${base_length/2} 0 0.115" rpy="0 0 0"/>
-  </joint>
-  <link name="lidar_link">
-    <visual>
-     <origin xyz="0 0 0" rpy="0 0 0"/>
-     <geometry>
-      <cylinder radius="0.0508" length="0.05"/>
-     </geometry>
-     <material name="Black">
-          <color rgba="${0/255} ${0/255} ${0/255} 1.0"/>
-     </material>
-    </visual>
-    <collision>
-     <origin xyz="0 0 0" rpy="0 0 0"/>
-     <geometry>
-      <cylinder radius="0.0508" length="0.05"/>
-     </geometry>
-    </collision>
     <inertial>
       <mass value="0.114" />
-      <origin xyz="0 0 0" rpy="0 0 0"/>
+      <origin xyz="0 0 0" rpy="0 0 0" />
       <inertia ixx="0.001" ixy="0" ixz="0" iyy="0.001" iyz="0" izz="0.001" />
     </inertial>
@@ -165,26 +216,26 @@
   <joint name="camera_joint" type="fixed">
     <axis xyz="0 1 0" />
-    <origin xyz="${base_length/2} 0 ${base_height}" rpy="0 0 0"/>
-    <parent link="map"/>
-    <child link="camera_link"/>
+    <origin xyz="${base_length/2} 0 ${base_height}" rpy="0 0 0" />
+    <parent link="base_link" />
+    <child link="camera_link" />
   </joint>
   <!-- Camera -->
   <link name="camera_link">
     <collision>
-      <origin xyz="0 0 0" rpy="0 0 0"/>
-      <geometry>
-    <box size="${camera} ${camera} ${camera}"/>
+      <origin xyz="0 0 0" rpy="0 0 0" />
+      <geometry>
+        <box size="${camera} ${camera} ${camera}" />
       </geometry>
     </collision>
     <visual>
-      <origin xyz="0 0 0" rpy="0 0 0"/>
-      <geometry>
-    <box size="${camera} ${camera} ${camera}"/>
-      </geometry>
-      <material name="red"/>
+      <origin xyz="0 0 0" rpy="0 0 0" />
+      <geometry>
+        <box size="${camera} ${camera} ${camera}" />
+      </geometry>
+      <material name="red" />
     </visual>
     <inertial>
       <mass value="1e-5" />
-      <origin xyz="0 0 0" rpy="0 0 0"/>
+      <origin xyz="0 0 0" rpy="0 0 0" />
       <inertia ixx="1e-6" ixy="0" ixz="0" iyy="1e-6" iyz="0" izz="1e-6" />
     </inertial>
@@ -230,9 +281,9 @@
         <distortion_p2>0.0</distortion_p2>
       </plugin>
-      <visualize>true</visualize>
+      <visualize>false</visualize>
     </sensor>
   </gazebo>
   <gazebo>
-  <!-- Differential drive -->
+    <!-- Differential drive -->
     <plugin name='diff_drive' filename='libgazebo_ros_diff_drive.so'>
       <!-- wheels -->
@@ -250,5 +301,5 @@
       <publish_wheel_tf>true</publish_wheel_tf>
       <odometry_frame>odom_demo</odometry_frame>
-      <robot_base_frame>map</robot_base_frame>
+      <robot_base_frame>base_link</robot_base_frame>
     </plugin>
   </gazebo>
@@ -303,5 +354,5 @@
         <frame_name>lidar_link</frame_name>
       </plugin>
-      <visualize>true</visualize>
+      <visualize>false</visualize>
     </sensor>
   </gazebo>

Commit message: modif color

File: robochon_description/urdf/robochon.urdf.xacro (robot description, xacro)
@@ -53,7 +53,4 @@
         <box size="${base_length} ${base_width} ${base_height}" />
       </geometry>
-      <material name="Cyan">
-        <color rgba="0 1.0 1.0 1.0" />
-      </material>
     </visual>
     <collision>
@@ -64,4 +61,7 @@
     <xacro:box_inertia m="15" w="${base_width}" d="${base_length}" h="${base_height}" />
   </link>
+  <gazebo reference="base_link">
+    <material>Gazebo/Grey</material>
+  </gazebo>
   <!-- Robot Footprint -->
   <link name="base_footprint" />
@@ -107,4 +107,9 @@
       <xacro:cylinder_inertia m="0.5" r="${wheel_radius}" h="${wheel_width}" />
     </link>
+    <gazebo reference="${prefix}_link">
+      <mu1>0.01</mu1>
+      <mu2>0.01</mu2>
+      <material>Gazebo/Grey</material>
+    </gazebo>
     <joint name="${prefix}_joint" type="continuous">
       <parent link="base_link" />
@@ -137,7 +142,4 @@
       <mu1>0.01</mu1>
       <mu2>0.01</mu2>
-      <visual>
-        <material>Gazebo/White</material>
-      </visual>
     </gazebo>
     <joint name="caster_joint_${prefix}" type="fixed">
@@ -149,4 +151,10 @@
   <xacro:front_caster prefix="front_left" link_daddy="base_link" y_reflect="1" />
   <xacro:front_caster prefix="front_right" link_daddy="base_link" y_reflect="-1" />
+  <gazebo reference="front_caster_front_left">
+    <material>Gazebo/Red</material>
+  </gazebo>
+  <gazebo reference="front_caster_front_right">
+    <material>Gazebo/Green</material>
+  </gazebo>
   <!-- Gripper -->
   <xacro:macro name="gripper" params="prefix x_reflect y_reflect z_reflect z_rotation lenght_x link_daddy">
@@ -157,7 +165,4 @@
           <box size="${gripper_length*lenght_x} ${gripper_width} ${gripper_height}" />
         </geometry>
-        <material name="Cyan">
-          <color rgba="0 1.0 1.0 1.0" />
-        </material>
       </visual>
       <collision>
@@ -171,7 +176,5 @@
       <mu1>1.4</mu1>
       <mu2>1.4</mu2>
-      <visual>
-        <material>Gazebo/White</material>
-      </visual>
+      <material>Gazebo/Grey</material>
     </gazebo>
     <joint name="${prefix}_joint" type="fixed">
@@ -233,5 +236,4 @@
         <box size="${camera} ${camera} ${camera}" />
       </geometry>
-      <material name="red" />
     </visual>
     <inertial>

Commit message: modfi urdf of

File: robochon_description/urdf/robochon.urdf.xacro (robot description, xacro)
@@ -53,4 +53,7 @@
         <box size="${base_length} ${base_width} ${base_height}" />
       </geometry>
+      <material name="Cyan">
+        <color rgba="0 1.0 1.0 1.0" />
+      </material>
     </visual>
     <collision>
@@ -62,5 +65,5 @@
   </link>
   <gazebo reference="base_link">
-    <material>Gazebo/Grey</material>
+    <material>Gazebo/Black</material>
   </gazebo>
   <!-- Robot Footprint -->
@@ -105,11 +108,9 @@
         </surface>
       </collision>
+      <gazebo reference="${prefix}_link">
+        <material>Gazebo/Grey</material>
+      </gazebo>
       <xacro:cylinder_inertia m="0.5" r="${wheel_radius}" h="${wheel_width}" />
     </link>
-    <gazebo reference="${prefix}_link">
-      <mu1>0.01</mu1>
-      <mu2>0.01</mu2>
-      <material>Gazebo/Grey</material>
-    </gazebo>
     <joint name="${prefix}_joint" type="continuous">
       <parent link="base_link" />
@@ -121,5 +122,4 @@
   <xacro:wheel prefix="drivewhl_l" x_reflect="-1" y_reflect="1" />
   <xacro:wheel prefix="drivewhl_r" x_reflect="-1" y_reflect="-1" />
-  <!-- Front caster -->
   <xacro:macro name="front_caster" params="prefix y_reflect link_daddy">
     <link name="front_caster_${prefix}">
@@ -147,5 +147,5 @@
       <parent link="${link_daddy}" />
       <child link="front_caster_${prefix}" />
-      <origin xyz="${caster_xoff} ${y_reflect*0.6*base_width/2} ${-(base_height/2)}" rpy="0 0 0" />
+      <origin xyz="${caster_xoff} ${y_reflect*0.7*base_width/2} ${-(base_height/2)}" rpy="0 0 0" />
     </joint>
   </xacro:macro>
@@ -166,4 +166,7 @@
           <box size="${gripper_length*lenght_x} ${gripper_width} ${gripper_height}" />
         </geometry>
+        <material name="Cyan">
+          <color rgba="0 1.0 1.0 1.0" />
+        </material>
       </visual>
       <collision>
@@ -185,6 +188,6 @@
     </joint>
   </xacro:macro>
-  <xacro:gripper prefix="gripper_l" x_reflect="1" y_reflect="1" z_reflect="1" z_rotation="0.15" lenght_x="1" link_daddy="base_link" />
-  <xacro:gripper prefix="gripper_r" x_reflect="1" y_reflect="-1" z_reflect="1" z_rotation="-0.15" lenght_x="1" link_daddy="base_link" />
+  <xacro:gripper prefix="gripper_l" x_reflect="1" y_reflect="1" z_reflect="1" z_rotation="0.3" lenght_x="1" link_daddy="base_link" />
+  <xacro:gripper prefix="gripper_r" x_reflect="1" y_reflect="-1" z_reflect="1" z_rotation="-0.3" lenght_x="1" link_daddy="base_link" />
   <xacro:gripper prefix="gripper_hor" x_reflect="-2" y_reflect="0" z_reflect="1" z_rotation="1.57" lenght_x="0.5" link_daddy="base_link" />
   <xacro:gripper prefix="gripper_l_front" x_reflect="1.7" y_reflect="-0.45" z_reflect="0" z_rotation="0.5" lenght_x="0.5" link_daddy="gripper_l_link" />
@@ -237,4 +240,5 @@
         <box size="${camera} ${camera} ${camera}" />
       </geometry>
+      <material name="red" />
     </visual>
     <inertial>

Commit message: urdf color ok

File: robochon_description/urdf/robochon.urdf.xacro (robot description, xacro)
@@ -65,5 +65,5 @@
   </link>
   <gazebo reference="base_link">
-    <material>Gazebo/Black</material>
+    <material>Gazebo/Grey</material>
   </gazebo>
   <!-- Robot Footprint -->
@@ -108,9 +108,9 @@
         </surface>
       </collision>
-      <gazebo reference="${prefix}_link">
-        <material>Gazebo/Grey</material>
-      </gazebo>
       <xacro:cylinder_inertia m="0.5" r="${wheel_radius}" h="${wheel_width}" />
     </link>
+    <gazebo reference="${prefix}_link">
+      <material>Gazebo/Grey</material>
+    </gazebo>
     <joint name="${prefix}_joint" type="continuous">
       <parent link="base_link" />
@@ -122,4 +122,5 @@
   <xacro:wheel prefix="drivewhl_l" x_reflect="-1" y_reflect="1" />
   <xacro:wheel prefix="drivewhl_r" x_reflect="-1" y_reflect="-1" />
+  <!-- Front caster -->
   <xacro:macro name="front_caster" params="prefix y_reflect link_daddy">
     <link name="front_caster_${prefix}">

Commit message: urdf size wheel ok

File: robochon_description/urdf/robochon.urdf.xacro (robot description, xacro)
@@ -148,5 +148,5 @@
       <parent link="${link_daddy}" />
       <child link="front_caster_${prefix}" />
-      <origin xyz="${caster_xoff} ${y_reflect*0.7*base_width/2} ${-(base_height/2)}" rpy="0 0 0" />
+      <origin xyz="${caster_xoff} ${y_reflect*0.6*base_width/2} ${-(base_height/2)}" rpy="0 0 0" />
     </joint>
   </xacro:macro>
