Commit message: modif size robot for color

File: robochon_description/urdf/robochon.urdf.xacro (robot description, xacro)
@@ -2,5 +2,5 @@
 <robot name="robochon" xmlns:xacro="http://ros.org/wiki/xacro">
   <!-- Define robot constants -->
-  <xacro:property name="base_width" value="${3*0.31}" />
+  <xacro:property name="base_width" value="${3.2*0.31}" />
   <xacro:property name="base_length" value="${3*0.42}" />
   <xacro:property name="base_height" value="0.18" />
@@ -148,5 +148,5 @@
       <parent link="${link_daddy}" />
       <child link="front_caster_${prefix}" />
-      <origin xyz="${caster_xoff} ${y_reflect*0.6*base_width/2} ${-(base_height/2)}" rpy="0 0 0" />
+      <origin xyz="${caster_xoff} ${y_reflect*0.55*base_width/2} ${-(base_height/2)}" rpy="0 0 0" />
     </joint>
   </xacro:macro>
@@ -192,6 +192,6 @@
   <xacro:gripper prefix="gripper_r" x_reflect="1" y_reflect="-1" z_reflect="1" z_rotation="-0.3" lenght_x="1" link_daddy="base_link" />
   <xacro:gripper prefix="gripper_hor" x_reflect="-2" y_reflect="0" z_reflect="1" z_rotation="1.57" lenght_x="0.5" link_daddy="base_link" />
-  <xacro:gripper prefix="gripper_l_front" x_reflect="1.7" y_reflect="-0.45" z_reflect="0" z_rotation="0.5" lenght_x="0.5" link_daddy="gripper_l_link" />
-  <xacro:gripper prefix="gripper_r_front" x_reflect="1.7" y_reflect="0.45" z_reflect="0" z_rotation="-0.5" lenght_x="0.5" link_daddy="gripper_r_link" />
+  <xacro:gripper prefix="gripper_l_front" x_reflect="1.7" y_reflect="-0.45" z_reflect="0" z_rotation="0.6" lenght_x="0.5" link_daddy="gripper_l_link" />
+  <xacro:gripper prefix="gripper_r_front" x_reflect="1.7" y_reflect="0.45" z_reflect="0" z_rotation="-0.6" lenght_x="0.5" link_daddy="gripper_r_link" />
   <!-- LIDAR -->
   <joint name="lidar_joint" type="fixed">

Commit message: final robot_description and control

File: robochon_description/urdf/robochon.urdf.xacro (robot description, xacro)
@@ -2,5 +2,5 @@
 <robot name="robochon" xmlns:xacro="http://ros.org/wiki/xacro">
   <!-- Define robot constants -->
-  <xacro:property name="base_width" value="${3.2*0.31}" />
+  <xacro:property name="base_width" value="${3*0.31}" />
   <xacro:property name="base_length" value="${3*0.42}" />
   <xacro:property name="base_height" value="0.18" />
@@ -148,5 +148,5 @@
       <parent link="${link_daddy}" />
       <child link="front_caster_${prefix}" />
-      <origin xyz="${caster_xoff} ${y_reflect*0.55*base_width/2} ${-(base_height/2)}" rpy="0 0 0" />
+      <origin xyz="${caster_xoff} ${y_reflect*0.7*base_width/2} ${-(base_height/2)}" rpy="0 0 0" />
     </joint>
   </xacro:macro>
@@ -192,6 +192,6 @@
   <xacro:gripper prefix="gripper_r" x_reflect="1" y_reflect="-1" z_reflect="1" z_rotation="-0.3" lenght_x="1" link_daddy="base_link" />
   <xacro:gripper prefix="gripper_hor" x_reflect="-2" y_reflect="0" z_reflect="1" z_rotation="1.57" lenght_x="0.5" link_daddy="base_link" />
-  <xacro:gripper prefix="gripper_l_front" x_reflect="1.7" y_reflect="-0.45" z_reflect="0" z_rotation="0.6" lenght_x="0.5" link_daddy="gripper_l_link" />
-  <xacro:gripper prefix="gripper_r_front" x_reflect="1.7" y_reflect="0.45" z_reflect="0" z_rotation="-0.6" lenght_x="0.5" link_daddy="gripper_r_link" />
+  <xacro:gripper prefix="gripper_l_front" x_reflect="1.7" y_reflect="-0.45" z_reflect="0" z_rotation="0.5" lenght_x="0.5" link_daddy="gripper_l_link" />
+  <xacro:gripper prefix="gripper_r_front" x_reflect="1.7" y_reflect="0.45" z_reflect="0" z_rotation="-0.5" lenght_x="0.5" link_daddy="gripper_r_link" />
   <!-- LIDAR -->
   <joint name="lidar_joint" type="fixed">
